Commit message: Adds position and velocity motion generators to FrankaHWSim
Features:
- This commit adds the 'hardware_interface/PositionJointInterface' and
'hardware_interface/VelocityJointInterface' interfaces to the
FrankaHWSim module. When a user chooses these interfaces, motion
generators (i.e. PID controllers) are used for controlling the robot.
- This commit adds the 'transmission' arg to the 'panda_arm.urdf.xacro'
file. By doing this, users now can set the hardware_interface that
is used in the panda arm joints when loading the 'panda_arm.urdf.xacro'
file.
- This commit adds the `effort_joint_trajectory_controller` and
`position_joint_trajectory_controller` controllers to the franka_gazebo
`sim_controllers.yaml` config.

File: franka_description/robots/panda_arm.urdf.xacro (robot description, xacro)
@@ -1,10 +1,9 @@
 <?xml version='1.0' encoding='utf-8'?>
 <robot xmlns:xacro="http://www.ros.org/wiki/xacro" name="panda">
-  <!-- Name of this panda -->
-  <xacro:arg name="arm_id" default="panda" />
-  <!-- Should a franka_gripper be mounted at the flange?" -->
-  <xacro:arg name="hand" default="false" />
-  <!-- Is the robot being simulated in gazebo?" -->
-  <xacro:arg name="gazebo" default="false" />
+  <xacro:arg name="arm_id" default="panda" /> <!-- Name of this panda -->
+  <xacro:arg name="hand"   default="false" /> <!-- Should a franka_gripper be mounted at the flange?" -->
+  <xacro:arg name="gazebo" default="false" /> <!-- Is the robot being simulated in gazebo?" -->
+  <xacro:arg name="transmission" default="hardware_interface/EffortJointInterface" /> <!-- The transmission that is used in the gazebo joints -->
+  <xacro:property name="arm_id" value="$(arg arm_id)" />
   <xacro:unless value="$(arg gazebo)">
     <!-- Create a URDF for a real hardware -->
@@ -35,11 +34,11 @@
       <child  link="$(arg arm_id)_link0" />
     </joint>
-    <xacro:gazebo-joint joint="$(arg arm_id)_joint1" transmission="hardware_interface/EffortJointInterface" />
-    <xacro:gazebo-joint joint="$(arg arm_id)_joint2" transmission="hardware_interface/EffortJointInterface" />
-    <xacro:gazebo-joint joint="$(arg arm_id)_joint3" transmission="hardware_interface/EffortJointInterface" />
-    <xacro:gazebo-joint joint="$(arg arm_id)_joint4" transmission="hardware_interface/EffortJointInterface" />
-    <xacro:gazebo-joint joint="$(arg arm_id)_joint5" transmission="hardware_interface/EffortJointInterface" />
-    <xacro:gazebo-joint joint="$(arg arm_id)_joint6" transmission="hardware_interface/EffortJointInterface" />
-    <xacro:gazebo-joint joint="$(arg arm_id)_joint7" transmission="hardware_interface/EffortJointInterface" />
+    <xacro:gazebo-joint joint="${arm_id}_joint1" transmission="$(arg transmission)" />
+    <xacro:gazebo-joint joint="${arm_id}_joint2" transmission="$(arg transmission)" />
+    <xacro:gazebo-joint joint="${arm_id}_joint3" transmission="$(arg transmission)" />
+    <xacro:gazebo-joint joint="${arm_id}_joint4" transmission="$(arg transmission)" />
+    <xacro:gazebo-joint joint="${arm_id}_joint5" transmission="$(arg transmission)" />
+    <xacro:gazebo-joint joint="${arm_id}_joint6" transmission="$(arg transmission)" />
+    <xacro:gazebo-joint joint="${arm_id}_joint7" transmission="$(arg transmission)" />
     <xacro:transmission-franka-state arm_id="$(arg arm_id)" />
     <xacro:transmission-franka-model arm_id="$(arg arm_id)"
