Commit message: Moves finger collision geometries to the finger joints
This commit moves the finger collision geometries to the finger joints.
This was done to prevent errors in third party libaries. Moveit for
example expects a collision geometry in each joint that can be
controlled.

File: franka_description/robots/hand.xacro (robot description, xacro)
@@ -41,12 +41,13 @@
         </geometry>
       </collision>
+    </link>
+    <link name="${ns}_leftfinger">
+      <visual>
+        <geometry>
+          <mesh filename="package://franka_description/meshes/visual/finger.dae"/>
+        </geometry>
+      </visual>
       <collision>
-        <origin xyz="0 0 0.1" rpy="0 ${pi/2} ${pi/2}"/>
-        <geometry>
-          <cylinder radius="${0.02+safety_distance}" length="0.1" />
-        </geometry>
-      </collision>
-      <collision>
-        <origin xyz="0 -0.05 0.1" rpy="0 0 0"/>
+        <origin xyz="0 0.01 0.0415" rpy="0 0 0"/>
         <geometry>
           <sphere radius="${0.02+safety_distance}"  />
@@ -54,7 +55,7 @@
       </collision>
       <collision>
-        <origin xyz="0 0.05 0.1" rpy="0 0 0"/>
+        <origin xyz="0 -0.015 0.0416" rpy="0 ${pi/2} ${pi/2}"/>
         <geometry>
-          <sphere radius="${0.02+safety_distance}"  />
+          <cylinder radius="${0.02+safety_distance}" length="0.05" />
         </geometry>
       </collision>
@@ -71,16 +72,4 @@
       <child link="${ns}_hand_tcp" />
     </joint>
-    <link name="${ns}_leftfinger">
-      <visual>
-        <geometry>
-          <mesh filename="package://franka_description/meshes/visual/finger.dae"/>
-        </geometry>
-      </visual>
-      <collision>
-        <geometry>
-          <mesh filename="package://franka_description/meshes/collision/finger.stl" />
-        </geometry>
-      </collision>
-    </link>
     <link name="${ns}_rightfinger">
       <visual>
@@ -91,7 +80,13 @@
       </visual>
       <collision>
-        <origin xyz="0 0 0" rpy="0 0 ${pi}" />
+        <origin xyz="0 -0.01 0.0415" rpy="0 0 0"/>
         <geometry>
-          <mesh filename="package://franka_description/meshes/collision/finger.stl" />
+          <sphere radius="${0.02+safety_distance}"  />
+        </geometry>
+      </collision>
+      <collision>
+        <origin xyz="0 0.015 0.0416" rpy="0 ${pi/2} ${pi/2}"/>
+        <geometry>
+          <cylinder radius="${0.02+safety_distance}" length="0.05" />
         </geometry>
       </collision>

Commit message: Define hand_tcp frame
... in the center between and aligned with the fingers

File: franka_description/robots/hand.xacro (robot description, xacro)
@@ -53,4 +53,11 @@
       </collision>
     </link>
+    <!-- Define the hand_tcp frame -->
+    <link name="${ns}_hand_tcp" />
+    <joint name="${ns}_hand_tcp_joint" type="fixed">
+      <origin xyz="0 0 0.1034" rpy="0 0 ${-pi/4}" />
+      <parent link="${ns}_hand" />
+      <child link="${ns}_hand_tcp" />
+    </joint>
     <link name="${ns}_leftfinger">
       <visual>
