Commit message: Fixes gazebo gripper action bug
This commit fixes a bug that was introduced by #147. In #147 the
finger collision geometries were replaced by more accurate meshes.
These more accurate messages however broke the 'gripper_action' action.
This commit migrates back to using geometries for the finger collision geometries.
The action server works fine when geometriesare used.

File: franka_description/robots/panda_gazebo.xacro (robot description, xacro)
@@ -292,6 +292,19 @@
       </visual>
       <collision>
-        <geometry>
-          <mesh filename="package://franka_description/meshes/collision/finger.stl" />
+        <origin xyz="0 0.0184 0.0101" rpy="0 0 0"/>
+        <geometry>
+          <box size="0.022 0.014 0.0177" />
+        </geometry>
+      </collision>
+      <collision>
+        <origin xyz="0 0.01655 0.02755" rpy="${3.257/(2*pi)} 0 0"/>
+        <geometry>
+          <box size="0.022 0.00686 0.0237" />
+        </geometry>
+      </collision>
+      <collision>
+        <origin xyz="0 0.0073 0.045" rpy="0 0 0"/>
+        <geometry>
+          <box size="0.022 0.0147 0.0178" />
         </geometry>
       </collision>
@@ -306,7 +319,19 @@
       </visual>
       <collision>
-        <origin xyz="0 0 0" rpy="0 0 ${pi}"/>
-        <geometry>
-          <mesh filename="package://franka_description/meshes/collision/finger.stl" />
+        <origin xyz="0 -0.0184 0.0101" rpy="0 0 0"/>
+        <geometry>
+          <box size="0.022 0.014 0.0177" />
+        </geometry>
+      </collision>
+      <collision>
+        <origin xyz="0 -0.01655 0.02755" rpy="${-3.257/(2*pi)} 0 0"/>
+        <geometry>
+          <box size="0.022 0.00686 0.0237" />
+        </geometry>
+      </collision>
+      <collision>
+        <origin xyz="0 -0.0073 0.045" rpy="0 0 0"/>
+        <geometry>
+          <box size="0.022 0.0147 0.0178" />
         </geometry>
       </collision>

Commit message: Define finger_joint2 as mimic joint of finger_joint1
Although, Gazebo doesn't support mimic joints natively,
FrankaHWSim does and MoveIt - for planning - should know
that the fingers will move in sync.

File: franka_description/robots/panda_gazebo.xacro (robot description, xacro)
@@ -325,4 +325,5 @@
       <axis xyz="0 -1 0"/>
       <limit effort="20" lower="0.0" upper="0.04" velocity="0.2"/>
+      <mimic joint="${ns}_finger_joint1" />
       <dynamics damping="0.3"/>
     </joint>

Commit message: Add hand_tcp frame to gazebo xacro.

File: franka_description/robots/panda_gazebo.xacro (robot description, xacro)
@@ -310,4 +310,11 @@
       </collision>
     </link>
+    <!-- Define the hand_tcp frame -->
+    <link name="${ns}_hand_tcp" />
+    <joint name="${ns}_hand_tcp_joint" type="fixed">
+      <origin xyz="0 0 0.1034" rpy="0 0 ${-pi/4}" />
+      <parent link="${ns}_hand" />
+      <child link="${ns}_hand_tcp" />
+    </joint>
     <link name="${ns}_rightfinger">
       <xacro:inertia-cylinder mass="15e-3" radius="0.01" h="0.04"/>

Commit message: fix: fix rha/develop merge conflicts
This commit fixes merged conflicts that were created by
def4a12ea3e08c3f09b4c4e0fc38e6252404e955.

File: franka_description/robots/panda_gazebo.xacro (robot description, xacro)
@@ -326,5 +326,5 @@
       <limit effort="20" lower="0.0" upper="0.04" velocity="0.2"/>
       <mimic joint="${ns}_finger_joint1" />
-      <dynamics damping="0.3"/>
+      <dynamics friction="0.0" damping="0.03"/>
     </joint>
   </xacro:macro>
